File: KiCad/M5Multimeter_v01/M5Multimeter.kicad_pcb (KiCad board)
At the start: 2 copper layers, 50 x 50 mm, 44 parts, among them J1 M-BUS, J10 INPUT1, J2 BAT, J20 INPUT2, Q10 BSS138, Q11 BSS138, Q20 BSS138, Q21 BSS138, SW1 SK-12D01-VG4

Commit message: GND / VCC pattern correction
Routing:
- net +3V3: track 27.4 -> 26.5 mm
Changed lines of the file:
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@@
     (thickness 1.6)
     (drawings 82)
-    (tracks 223)
+    (tracks 221)
     (zones 0)
     (modules 44)
@@
     (44 Edge.Cuts user)
     (45 Margin user)
-    (46 B.CrtYd user)
-    (47 F.CrtYd user)
+    (46 B.CrtYd user hide)
+    (47 F.CrtYd user hide)
     (48 B.Fab user hide)
     (49 F.Fab user hide)
@@
     (aux_axis_origin 104 133)
     (grid_origin 104 133)
-    (visible_elements 7FFFFFFF)
+    (visible_elements 7FFFFF7F)
     (pcbplotparams
       (layerselection 0x010f0_ffffffff)
@@
     (tags SOD-323)
     (attr smd)
-    (fp_text reference D20 (at 0 1.778 90) (layer F.SilkS)
+    (fp_text reference D20 (at 0.132 -2.03 90) (layer F.SilkS)
       (effects (font (size 1 1) (thickness 0.15)))
     )
@@
     (tags SOD-323)
     (attr smd)
-    (fp_text reference D21 (at 2.54 -1.778 90) (layer F.SilkS)
+    (fp_text reference D21 (at 3.076 -0.78 90) (layer F.SilkS)
       (effects (font (size 1 1) (thickness 0.15)))
     )
@@
     (tags "resistor 0603")
     (attr smd)
-    (fp_text reference R20 (at 0 -1.45 180) (layer F.SilkS)
+    (fp_text reference R20 (at 0.286 1.652 180) (layer F.SilkS)
       (effects (font (size 1 1) (thickness 0.15)))
     )
@@
     (tags "resistor 0603")
     (attr smd)
-    (fp_text reference R21 (at 0 -1.45 270) (layer F.SilkS)
+    (fp_text reference R21 (at -2.822 -0.188 270) (layer F.SilkS)
       (effects (font (size 1 1) (thickness 0.15)))
     )
@@
     (tags "resistor 0603")
     (attr smd)
-    (fp_text reference R24 (at 2.794 0 270) (layer F.SilkS)
+    (fp_text reference R24 (at -0.132 1.488 270) (layer F.SilkS)
       (effects (font (size 1 1) (thickness 0.15)))
     )
@@
     (tags "resistor 0603")
     (attr smd)
-    (fp_text reference R26 (at -2.794 0) (layer F.SilkS)
+    (fp_text reference R26 (at -0.122 -1.532) (layer F.SilkS)
       (effects (font (size 1 1) (thickness 0.15)))
     )
@@
     (tags "resistor 0603")
     (attr smd)
-    (fp_text reference R27 (at -2.794 0 90) (layer F.SilkS)
+    (fp_text reference R27 (at 3.072 0 90) (layer F.SilkS)
       (effects (font (size 1 1) (thickness 0.15)))
     )
@@
     (tags "resistor 0603")
     (attr smd)
-    (fp_text reference R28 (at 3.048 0) (layer F.SilkS)
+    (fp_text reference R28 (at 0.012 -1.532) (layer F.SilkS)
       (effects (font (size 1 1) (thickness 0.15)))
     )
@@
   (segment (start 121.305 110.682) (end 121.271 110.648) (width 0.25) (layer F.Cu) (net 13))
   (segment (start 121.78 110.682) (end 121.305 110.682) (width 0.5) (layer F.Cu) (net 13) (status 10))
-  (segment (start 121.271 110.648) (end 116.7 110.648) (width 0.5) (layer F.Cu) (net 13))
-  (segment (start 116.7 110.648) (end 116.192 110.14) (width 0.5) (layer F.Cu) (net 13))
+  (segment (start 121.271 110.648) (end 116.7 110.648) (width 1) (layer F.Cu) (net 13))
+  (segment (start 116.7 110.648) (end 116.192 110.14) (width 1) (layer F.Cu) (net 13))
   (via (at 115.938 103.028) (size 0.6) (drill 0.4) (layers F.Cu B.Cu) (net 13))
   (segment (start 116.192 110.14) (end 115.938 109.886) (width 0.5) (layer F.Cu) (net 13))
-  (segment (start 115.938 109.886) (end 115.938 103.028) (width 0.5) (layer F.Cu) (net 13))
+  (segment (start 115.938 109.886) (end 115.938 103.028) (width 1) (layer F.Cu) (net 13))
   (segment (start 113.283 103.028) (end 113.175 102.92) (width 0.25) (layer B.Cu) (net 13) (status 30))
-  (segment (start 115.938 103.028) (end 113.283 103.028) (width 0.5) (layer B.Cu) (net 13) (status 20))
-  (segment (start 122.034 99.798) (end 122.034 98.998) (width 0.5) (layer F.Cu) (net 13) (status 20))
-  (segment (start 113.175 102.92) (end 114.268 102.92) (width 0.5) (layer F.Cu) (net 13) (status 10))
-  (segment (start 114.268 102.92) (end 114.62099 102.56701) (width 0.5) (layer F.Cu) (net 13))
-  (segment (start 114.62099 102.56701) (end 114.62099 101.528108) (width 0.5) (layer F.Cu) (net 13))
-  (segment (start 114.62099 101.528108) (end 116.042098 100.107) (width 0.5) (layer F.Cu) (net 13))
-  (segment (start 116.042098 100.107) (end 121.725 100.107) (width 0.5) (layer F.Cu) (net 13))
-  (segment (start 121.725 100.107) (end 122.034 99.798) (width 0.5) (layer F.Cu) (net 13))
+  (segment (start 115.938 103.028) (end 113.283 103.028) (width 1) (layer B.Cu) (net 13) (status 20))
+  (segment (start 115.75 100.25) (end 113.175 102.92) (width 1) (layer F.Cu) (net 13))
+  (segment (start 116.25 99.75) (end 115.75 100.25) (width 1) (layer F.Cu) (net 13))
+  (segment (start 121.5 99.75) (end 116.25 99.75) (width 1) (layer F.Cu) (net 13))
+  (segment (start 122.034 98.998) (end 122.034 99.216) (width 1) (layer F.Cu) (net 13))
+  (segment (start 122.034 99.216) (end 121.5 99.75) (width 1) (layer F.Cu) (net 13))
   (segment (start 118.388 127.388) (end 119 128) (width 1) (layer F.Cu) (net 21) (status 30))
   (segment (start 116.7 127.388) (end 118.388 127.388) (width 1) (layer F.Cu) (net 21) (status 30))
@@
   (segment (start 109.892 114.458) (end 108.73 115.62) (width 0.25) (layer B.Cu) (net 25) (status 20))
   (segment (start 113.801002 114.458) (end 109.892 114.458) (width 0.25) (layer B.Cu) (net 25))
-  (segment (start 138.095001 99.912001) (end 137.265002 100.742) (width 0.25) (layer F.Cu) (net 26))
-  (segment (start 138.095001 97.614999) (end 138.095001 99.912001) (width 0.25) (layer F.Cu) (net 26))
-  (segment (start 139.56 95.65) (end 139.56 96.15) (width 0.25) (layer F.Cu) (net 26) (status 10))
+  (segment (start 114.522 108) (end 113.175 108) (width 0.25) (layer F.Cu) (net 26))
+  (segment (start 115.001116 107.520884) (end 114.522 108) (width 0.25) (layer F.Cu) (net 26))
+  (segment (start 115.001116 102.23234) (end 115.001116 107.520884) (width 0.25) (layer F.Cu) (net 26))
   (segment (start 139.56 96.15) (end 138.095001 97.614999) (width 0.25) (layer F.Cu) (net 26))
-  (segment (start 137.265002 100.742) (end 116.192 100.742) (width 0.25) (layer F.Cu) (net 26))
-  (segment (start 116.192 100.742) (end 115.176 101.758) (width 0.25) (layer F.Cu) (net 26))
-  (segment (start 115.176 101.758) (end 115.176 107.346) (width 0.25) (layer F.Cu) (net 26))
-  (segment (start 114.522 108) (end 113.175 108) (width 0.25) (layer F.Cu) (net 26) (status 20))
-  (segment (start 115.176 107.346) (end 114.522 108) (width 0.25) (layer F.Cu) (net 26))
+  (segment (start 139.56 95.65) (end 139.56 96.15) (width 0.25) (layer F.Cu) (net 26))
+  (segment (start 138.095001 97.614999) (end 138.095001 99.912001) (width 0.25) (layer F.Cu) (net 26))
+  (segment (start 138.095001 99.912001) (end 137.265002 100.742) (width 0.25) (layer F.Cu) (net 26))
+  (segment (start 137.265002 100.742) (end 116.491456 100.742) (width 0.25) (layer F.Cu) (net 26))
+  (segment (start 116.491456 100.742) (end 115.001116 102.23234) (width 0.25) (layer F.Cu) (net 26))
   (segment (start 131.686 98.202) (end 131.686 100.488) (width 0.25) (layer B.Cu) (net 27))
   (segment (start 131.686 100.488) (end 130.162 102.012) (width 0.25) (layer B.Cu) (net 27))
